Commit message: fix: elspider air gazebo sim

File: legged_examples/legged_hexapod/legged_hexapod_description/urdf/gazebo.xacro (robot description, xacro)
@@ -2,8 +2,27 @@
 <robot xmlns:xacro="http://ros.org/wiki/xacro">
     <!-- ros_control plugin -->
-    <gazebo>
+    <!-- <gazebo>
         <plugin name="gazebo_ros_control" filename="libgazebo_ros_control.so">
             <robotNamespace>/elspider_air</robotNamespace>
             <robotSimType>gazebo_ros_control/DefaultRobotHWSim</robotSimType>
+        </plugin>
+    </gazebo> -->
+    <gazebo>
+        <plugin name="gazebo_ros_control" filename="liblegged_hw_sim.so">
+            <robotNamespace>/</robotNamespace>
+            <robotParam>legged_robot_description</robotParam>
+            <robotSimType>legged_gazebo/LeggedHWSim</robotSimType>
+        </plugin>
+    </gazebo>
+    <gazebo>
+        <plugin name="p3d_base_controller" filename="libgazebo_ros_p3d.so">
+            <alwaysOn>true</alwaysOn>
+            <updateRate>1000.0</updateRate>
+            <bodyName>base</bodyName>
+            <topicName>ground_truth/state</topicName>
+            <gaussianNoise>0</gaussianNoise>
+            <frameName>world</frameName>
+            <xyzOffsets>0 0 0</xyzOffsets>
+            <rpyOffsets>0 0 0</rpyOffsets>
         </plugin>
     </gazebo>
@@ -20,5 +39,5 @@
     </gazebo>
     <!-- simulates a 6 dof position and rate sensor -->
-    <gazebo>
+    <!-- <gazebo>
         <plugin name="p3d" filename="libgazebo_ros_p3d.so">
             <alwaysOn>true</alwaysOn>
@@ -28,7 +47,7 @@
             <frameName>world</frameName>
         </plugin>
-    </gazebo>
+    </gazebo> -->
     <!-- imu plugin -->
-    <gazebo reference="${ns}imu_link">
+    <!-- <gazebo reference="${ns}imu_link">
         <gravity>true</gravity>
         <sensor name="imu_sensor" type="imu">
@@ -48,5 +67,5 @@
             <pose>0 0 0 0 0 0</pose>
         </sensor>
-    </gazebo>
+    </gazebo> -->
     <!-- camera plugin -->
     <!-- <xacro:include filename="$(find realsense_ros_gazebo)/xacro/tracker.xacro"/>

File: legged_examples/legged_hexapod/legged_hexapod_description/urdf/leg.xacro (robot description, xacro)
@@ -168,4 +168,5 @@
             <mu2>0.2</mu2>
             <self_collide>1</self_collide>
+            <material>Gazebo/DarkGrey</material>
         </gazebo>
         <gazebo reference="${ns}${name}_THIGH">
@@ -173,4 +174,5 @@
             <mu2>0.2</mu2>
             <self_collide>1</self_collide>
+            <material>Gazebo/DarkGrey</material>
         </gazebo>
         <gazebo reference="{name}_SHANK">
@@ -178,4 +180,5 @@
             <mu2>0.2</mu2>
             <self_collide>1</self_collide>
+            <material>Gazebo/DarkGrey</material>
         </gazebo>
         <gazebo reference="${ns}${name}_FOOT">
@@ -188,4 +191,5 @@
             <kp value="20.0"/>
             <kd value="10.0"/>
+            <material>Gazebo/DarkGrey</material>
         </gazebo>
     </xacro:macro>

File: legged_examples/legged_hexapod/legged_hexapod_description/urdf/robot.xacro (robot description, xacro)
@@ -13,4 +13,5 @@
     <xacro:include filename="$(find legged_hexapod_description)/urdf/trunk.xacro"/>
     <xacro:include filename="$(find legged_hexapod_description)/urdf/leg.xacro"/>
+    <xacro:include filename="$(find legged_hexapod_description)/urdf/imu.xacro"/>
     <xacro:include filename="$(find legged_hexapod_description)/urdf/gazebo.xacro"/>
     <xacro:if value="${sensor_module_name == 'HexPercept1'}">
@@ -32,4 +33,5 @@
         </xacro:HexPercept3>
     </xacro:if>
+    <xacro:IMU connected_to="base" imu_name="base_imu" xyz="0. 0. 0." rpy="0. 0. 0."/>
     <xacro:leg name="aRF" mirror="1" back = "1" special = "1" special2 = "1">
         <origin rpy="0 -0 0" xyz="0.3 -0.08 0.011"/>
